File: profielWerkstuk.kicad_sch (KiCad schematic)
At the start: 138 parts, among them Q1 BF981, Q2 2N5179, SW1 SW_HF/VHF, SW2 SW_ANT, SW3 SW_PRESELECT_HFa, SW4 SW_PRESELECT_VHFa, SW5 SW_PRESELECT_HFb, SW6 SW_PRESELECT_VHFb, T1 Transformer_1P_SS, T10 Transformer_1P_SS, T11 Transformer_1P_SS, T12 Transformer_1P_SS, T2 Transformer_1P_SS, T3 Transformer_1P_SS, T4 Transformer_1P_SS, T5 Transformer_1P_SS, T6 1:5 winding, T8 Transformer_1P_SS, T9 Transformer_1P_SS

Commit message: worked on amp
Parts:
- added C40: 1-10p, symbol Device:C_Trim
- added C42: 200p, symbol Device:C
- added C43: 10n, symbol Device:C
- added C44: 5-30p, symbol Device:C_Trim
- added C45: 1n, symbol Device:C
- added FB1, FB2, FB3: (no value), symbol Device:FerriteBead_Small
- added L37: 56n, symbol Device:L
- added R21: 100, symbol Device:R
- added R22: 100k, symbol Device:R
- added R23: 47k, symbol Device:R
- added R24: 22, symbol Device:R
- added T7: 5:1 winding, symbol Device:Transformer_1P_1S
Connections:
- net GNDREF: now also C43.2, C45.2, R21.1, R22.1, T7.2 (AB), T7.3 (SA)
- net at Q1.1 (S): now also R21.2; no longer XF1.3 (out)
- net at Q1.2 (D): now also C42.1, C44.2, L37.1, T7.1 (AA)
- net at Q1.3 (G2): now also C43.1, FB1.2
- net at Q1.4 (G1): now also R24.2
- net at T9.1 (AA): now also T7.4 (SB)
- new net: C42.2, C44.1, C45.1, FB3.2, L37.2
- new net: FB1.1, R23.1
- new net: FB2.2, R23.2
- new net: C40.2, R22.2, R24.1
- new net: C40.1, XF1.3 (out)
Other:
- note added: "put AGC here -->"
- note added: "put VCC here -->"
- moved on the sheet: C35, C36, C37, C38, D20, D21, D22, D23, D24, D25, D26, D27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
