File: highRangeCircuit/profielWerkstuk.kicad_sch (KiCad schematic)
At the start: 152 parts, among them Q1 BF981, Q2 2N5179, SW1 SW_HF/VHF, SW2 SW_ANT, SW3 SW_PRESELECT_HFa, SW4 SW_PRESELECT_VHFa, SW5 SW_PRESELECT_HFb, SW6 SW_PRESELECT_VHFb, T1 Transformer_1P_SS, T10 Transformer_1P_SS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

Commit message: moved some stuff and started with new preselectors
Parts:
- removed C40: 1-10p, symbol Device:C_Trim
- removed C42: 200p, symbol Device:C
- removed C43: 10n, symbol Device:C
- removed C44: 5-30p, symbol Device:C_Trim
- removed C45: 1n, symbol Device:C
- removed FB1, FB2, FB3: (no value), symbol Device:FerriteBead_Small
- removed L37: 56n, symbol Device:L
- removed Q2: 2N5179, symbol Transistor_BJT:Q_NPN_BCE
- removed R21: 100, symbol Device:R
- removed R22: 100k, symbol Device:R
- removed R23: 47k, symbol Device:R
- removed R24: 22, symbol Device:R
- added Q1: 2N5770, symbol Transistor_BJT:Q_NPN_BCE
- added SW7: SW_PRESELECT_HFc, symbol Switch:SW_Rotary_1x4_MP
- added SW8: SW_PRESELECT_HFd, symbol Switch:SW_Rotary_1x4_MP
Connections:
- net at T1.1 (AA): now also SW7.5
- net at Q1.2 (D): no longer T7.1 (AA)
Other:
- note added: "1st IF: HF: 45 MHz VHF 70 MHz"
- note added: "1st LO: HF: 47 - 77 MHz VHF 45 MHz"
- note removed: "1st IF: HF: 10.7 MHz VHF 45 MHz"
- note removed: "put AGC here -->"
- note removed: "put VCC here -->"
- moved on the sheet: C35, C36, C37, C38, D20, D21, D22, D23, D24, D25, D26, D27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
