File: AM-Receiver/AM-Receiver.kicad_sch (KiCad schematic)
At the start: 9 parts

Commit message: needs some more tuning
Parts:
- added Q1: 2N3904, Package_TO_SOT_THT:TO-92_Inline, symbol Transistor_BJT:2N3904
Other:
- moved on the sheet: C3, L2
Changed lines of the file:
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@@
 	(paper "A4")
 	(junction
-		(at 113.03 53.34)
+		(at 87.63 63.5)
 		(diameter 0)
 		(color 0 0 0 0)
 	)
 	(junction
-		(at 113.03 60.96)
+		(at 111.76 50.8)
 		(diameter 0)
 		(color 0 0 0 0)
@@
 	)
 	(junction
-		(at 113.03 50.8)
+		(at 111.76 53.34)
+		(diameter 0)
+		(color 0 0 0 0)
+	)
+	(junction
+		(at 111.76 60.96)
 		(diameter 0)
 		(color 0 0 0 0)
@@
 	)
 	(junction
-		(at 87.63 63.5)
-		(diameter 0)
-		(color 0 0 0 0)
-	)
-	(junction
 		(at 46.99 50.8)
 		(diameter 0)
@@
 	(wire
 		(pts
+			(xy 111.76 50.8) (xy 125.73 50.8)
+		)
+		(stroke
+			(width 0)
+			(type default)
+		)
+	)
+	(wire
+		(pts
 			(xy 87.63 50.8) (xy 87.63 53.34)
 		)
@@
 	(wire
 		(pts
-			(xy 87.63 63.5) (xy 113.03 63.5)
-		)
-		(stroke
-			(width 0)
-			(type default)
-		)
-	)
-	(wire
-		(pts
-			(xy 113.03 50.8) (xy 113.03 53.34)
-		)
-		(stroke
-			(width 0)
-			(type default)
-		)
-	)
-	(wire
-		(pts
-			(xy 113.03 53.34) (xy 116.84 53.34)
+			(xy 87.63 63.5) (xy 111.76 63.5)
+		)
+		(stroke
+			(width 0)
+			(type default)
+		)
+	)
+	(wire
+		(pts
+			(xy 111.76 50.8) (xy 111.76 53.34)
 		)
 		(stroke
@@
 	(wire
 		(pts
-			(xy 113.03 50.8) (xy 125.73 50.8)
-		)
-		(stroke
-			(width 0)
-			(type default)
-		)
-	)
-	(wire
-		(pts
 			(xy 46.99 58.42) (xy 59.69 58.42)
 		)
@@
 	(wire
 		(pts
-			(xy 104.14 50.8) (xy 113.03 50.8)
+			(xy 104.14 50.8) (xy 111.76 50.8)
 		)
 		(stroke
@@
 	(wire
 		(pts
+			(xy 111.76 53.34) (xy 115.57 53.34)
+		)
+		(stroke
+			(width 0)
+			(type default)
+		)
+	)
+	(wire
+		(pts
 			(xy 87.63 60.96) (xy 91.44 60.96)
 		)
@@
 	(wire
 		(pts
-			(xy 113.03 60.96) (xy 113.03 63.5)
-		)
-		(stroke
-			(width 0)
-			(type default)
-		)
-	)
-	(wire
-		(pts
-			(xy 110.49 60.96) (xy 113.03 60.96)
+			(xy 111.76 60.96) (xy 111.76 63.5)
+		)
+		(stroke
+			(width 0)
+			(type default)
+		)
+	)
+	(wire
+		(pts
+			(xy 109.22 60.96) (xy 111.76 60.96)
 		)
 		(stroke
@@
 	(wire
 		(pts
-			(xy 110.49 53.34) (xy 113.03 53.34)
+			(xy 109.22 53.34) (xy 111.76 53.34)
 		)
 		(stroke
@@
 	(wire
 		(pts
-			(xy 113.03 60.96) (xy 116.84 60.96)
+			(xy 111.76 60.96) (xy 115.57 60.96)
 		)
 		(stroke
@@
 	)
 	(symbol
+		(lib_id "Transistor_BJT:2N3904")
+		(at 123.19 102.87 0)
+		(unit 1)
+		(body_style 1)
+		(exclude_from_sim no)
+		(in_bom yes)
+		(on_board yes)
+		(in_pos_files yes)
+		(dnp no)
+		(fields_autoplaced yes)
+		(property "Reference" "Q1"
+			(at 128.27 101.5999 0)
+			(show_name no)
+			(do_not_autoplace no)
+			(effects
+				(font
+					(size 1.27 1.27)
+				)
+				(justify left)
+			)
+		)
+		(property "Value" "2N3904"
+			(at 128.27 104.1399 0)
+			(show_name no)
+			(do_not_autoplace no)
+			(effects
+				(font
+					(size 1.27 1.27)
+				)
+				(justify left)
+			)
+		)
+		(property "Footprint" "Package_TO_SOT_THT:TO-92_Inline"
+			(at 128.27 104.775 0)
+			(hide yes)
+			(show_name no)
+			(do_not_autoplace no)
+			(effects
+				(font
+					(size 1.27 1.27)
+					(italic yes)
+				)
+				(justify left)
+			)
+		)
+		(property "Datasheet" "https://www.onsemi.com/pub/Collateral/2N3903-D.PDF"
+			(at 123.19 102.87 0)
+			(hide yes)
+			(show_name no)
+			(do_not_autoplace no)
+			(effects
+				(font
+					(size 1.27 1.27)
+				)
+				(justify left)
+			)
+		)
+		(property "Description" "0.2A Ic, 40V Vce, Small Signal NPN Transistor, TO-92"
+			(at 123.19 102.87 0)
+			(hide yes)
+			(show_name no)
+			(do_not_autoplace no)
+			(effects
+				(font
+					(size 1.27 1.27)
+				)
+			)
+		)
+		(property "Sim.Device" "NPN"
+			(at 123.19 102.87 0)
+			(hide yes)
+			(show_name no)
+			(do_not_autoplace no)
+			(effects
+				(font
+					(size 1.27 1.27)
+				)
+			)
+		)
+		(property "Sim.Pins" "1=E 2=B 3=C"
+			(at 123.19 102.87 0)
+			(hide yes)
+			(show_name no)
+			(do_not_autoplace no)
+			(effects
+				(font
+					(size 1.27 1.27)
+				)
+			)
+		)
+		(pin "2"
+		)
+		(pin "3"
+		)
+		(pin "1"
+		)
+		(instances
+			(project "AM-Receiver"
+				(path "/8ed7e543-7d50-486c-b61b-ae9d489b8386"
+					(reference "Q1")
+					(unit 1)
+				)
+			)
+		)
+	)
+	(symbol
 		(lib_id "Device:L")
-		(at 116.84 57.15 0)
+		(at 115.57 57.15 0)
 		(unit 1)
 		(body_style 1)
@@
 		(fields_autoplaced yes)
 		(property "Reference" "L2"
-			(at 118.11 55.8799 0)
+			(at 116.84 55.8799 0)
 			(show_name no)
 			(do_not_autoplace no)
@@
 		)
 		(property "Value" "80u"
-			(at 118.11 58.4199 0)
+			(at 116.84 58.4199 0)
 			(show_name no)
 			(do_not_autoplace no)
@@
 		)
 		(property "Footprint" ""
-			(at 116.84 57.15 0)
+			(at 115.57 57.15 0)
 			(hide yes)
 			(show_name no)
@@
 		)
 		(property "Datasheet" ""
-			(at 116.84 57.15 0)
+			(at 115.57 57.15 0)
 			(hide yes)
 			(show_name no)
@@
 		)
 		(property "Description" "Inductor"
-			(at 116.84 57.15 0)
+			(at 115.57 57.15 0)
 			(hide yes)
 			(show_name no)
@@
 	(symbol
 		(lib_id "Device:C_Variable")
-		(at 110.49 57.15 0)
+		(at 109.22 57.15 0)
 		(unit 1)
 		(body_style 1)
@@
 		(dnp no)
 		(property "Reference" "C3"
-			(at 105.41 56.134 0)
+			(at 104.14 56.134 0)
 			(show_name no)
 			(do_not_autoplace no)
@@
 		)
 		(property "Value" "60p-140p"
-			(at 98.806 58.928 0)
+			(at 97.536 58.928 0)
 			(show_name no)
 			(do_not_autoplace no)
@@
 		)
 		(property "Footprint" ""
-			(at 110.49 57.15 0)
+			(at 109.22 57.15 0)
 			(hide yes)
 			(show_name no)
@@
 		)
 		(property "Datasheet" ""
-			(at 110.49 57.15 0)
+			(at 109.22 57.15 0)
 			(hide yes)
 			(show_name no)
@@
 		)
 		(property "Description" "Variable capacitor"
-			(at 110.49 57.15 0)
-			(hide yes)
-			(show_name no)
+			(at 109.22 57.15 0)
+			(hide yes)
+			(show_name no)
